Commit message: add obj and mtl file, change path to mtl, change dae path to obj path

File: urdf/arm/openarm_macro.xacro (robot description, xacro)
@@ -27,5 +27,5 @@
         <xacro:openarm-kinematics-link config="${kinematics_link}" name="${name}" />
         <geometry>
-          <mesh filename="package://${description_pkg}/meshes/arm/${arm_type}/visual/${name}.dae" scale="0.001 ${0.001*reflect} 0.001" />
+          <mesh filename="package://${description_pkg}/meshes/arm/${arm_type}/visual/${name}.obj" scale="0.001 ${0.001*reflect} 0.001" />
         </geometry>
       </visual>

File: urdf/ee/openarm_hand.xacro (robot description, xacro)
@@ -29,5 +29,5 @@
         <xacro:openarm-ee-kinematics-link config="${ee_kinematics_link}" name="left_finger" />
         <geometry>
-          <mesh filename="package://${description_pkg}/meshes/ee/${ee_type}/visual/finger.dae" scale="0.001 0.001 0.001"/>
+          <mesh filename="package://${description_pkg}/meshes/ee/${ee_type}/visual/finger.obj" scale="0.001 0.001 0.001"/>
         </geometry>
       </visual>
@@ -44,5 +44,5 @@
         <xacro:openarm-ee-kinematics-link config="${ee_kinematics_link}" name="right_finger" />
         <geometry>
-          <mesh filename="package://${description_pkg}/meshes/ee/${ee_type}/visual/finger.dae" scale="0.001 -0.001 0.001"/>
+          <mesh filename="package://${description_pkg}/meshes/ee/${ee_type}/visual/finger.obj" scale="0.001 -0.001 0.001"/>
         </geometry>
       </visual>

File: urdf/ee/openarm_hand_macro.xacro (robot description, xacro)
@@ -25,5 +25,5 @@
         <xacro:openarm-ee-kinematics-link config="${ee_kinematics_link}" name="${name}" />
         <geometry>
-          <mesh filename="package://${description_pkg}/meshes/ee/${ee_type}/visual/${name}.dae" scale="0.001 0.001 0.001" />
+          <mesh filename="package://${description_pkg}/meshes/ee/${ee_type}/visual/${name}.obj" scale="0.001 0.001 0.001" />
         </geometry>
       </visual>
